Commit message: [envs/isaac] Set different sim params for envs.

File: multimodal_robot_model/envs/assets/isaac/objects/cabinet/cabinet.urdf (robot description, URDF)
Before this commit: robot cabinet, 7 links, 6 joints
Joints:
- joint door: origin xyz=0.0 0.1 0.305 -> xyz=0.0 0.101 0.306

Commit message: [envs/assets] Update color of cabinet.

File: multimodal_robot_model/envs/assets/isaac/objects/cabinet/cabinet.urdf (robot description, URDF)
Before this commit: robot cabinet, 7 links, 6 joints
Links:
- link wall1: geometry collision box size=0.13 0.01 0.25; visual box size=0.13 0.01 0.25
