Commit message: [envs] Update aloha env.

File: multimodal_robot_model/envs/assets/common/robots/aloha/vx300s.urdf (robot description, URDF)
Before this commit: robot vx300s, 14 links, 13 joints
Joints:
- joint gripper: type continuous -> fixed
- joint left_finger: type prismatic -> fixed
- joint right_finger: type prismatic -> fixed
